File: TacTile-A/TacTile-A.kicad_sch (KiCad schematic)
At the start: 92 parts, among them J1 Conn_01x01, J2 Conn_01x01, J3 Conn_01x01, J4 Conn_01x01, U1 MCP14A0303xMNY, U2 MCP14A0303xMNY, U3 MCP14A0303xMNY, U4 MCP14A0303xMNY, U5 MCP14A0303xMNY, U6 MCP14A0303xMNY, U7 MCP14A0303xMNY, U8 MCP14A0303xMNY

Commit message: Added voltage input to A MOSFETs
Parts:
- added JMP17: ~, TacTile:Jumper_Connect, symbol TacTile:Jumper_Connect
Connections:
- net GND10: now also U6.5 (~{OUTB}); no longer U6.7 (~{OUTA})
- net GND11: now also U6.7 (~{OUTA}); no longer U6.5 (~{OUTB})
- net GND12: now also U7.5 (~{OUTB}); no longer U7.7 (~{OUTA})
- net GND13: now also U7.7 (~{OUTA}); no longer U7.5 (~{OUTB})
- net GND14: now also U8.5 (~{OUTB}); no longer U8.7 (~{OUTA})
- net GND15: now also U8.7 (~{OUTA}); no longer U8.5 (~{OUTB})
- net GND8: now also U5.5 (~{OUTB}); no longer U5.7 (~{OUTA})
- net GND9: now also U5.7 (~{OUTA}); no longer U5.5 (~{OUTB})
- net INP10: now also U6.4 (INB); no longer U6.2 (INA)
- net INP11: now also U6.2 (INA); no longer U6.4 (INB)
- net INP12: now also U7.4 (INB); no longer U7.2 (INA)
- net INP13: now also U7.2 (INA); no longer U7.4 (INB)
- net INP14: now also U8.4 (INB); no longer U8.2 (INA)
- net INP15: now also U8.2 (INA); no longer U8.4 (INB)
- net INP8: now also U5.4 (INB); no longer U5.2 (INA)
- net INP9: now also U5.2 (INA); no longer U5.4 (INB)
- net VCC: now reaches U8.6 (V+)
- net VCC: now also U1.6 (V+), U2.6 (V+), U3.6 (V+), U4.6 (V+), U5.6 (V+), U6.6 (V+), U7.6 (V+), JMP17.1 (A)
Changed lines of the file:
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@@
     (effects (font (size 1.27 1.27)) (justify left bottom))
   )
-  (label "GND15" (at 186.69 96.52 0) (fields_autoplaced)
+  (label "GND15" (at 186.69 91.44 0) (fields_autoplaced)
     (effects (font (size 1.27 1.27)) (justify left bottom))
   )
@@
     (effects (font (size 1.27 1.27)) (justify left bottom))
   )
-  (label "GND14" (at 186.69 91.44 0) (fields_autoplaced)
+  (label "GND14" (at 186.69 96.52 0) (fields_autoplaced)
     (effects (font (size 1.27 1.27)) (justify left bottom))
   )
@@
     (effects (font (size 1.27 1.27)) (justify left bottom))
   )
+  (label "VCC" (at 176.53 60.96 0) (fields_autoplaced)
+    (effects (font (size 1.27 1.27)) (justify left bottom))
+  )
   (label "GND5" (at 125.73 85.09 0) (fields_autoplaced)
     (effects (font (size 1.27 1.27)) (justify left bottom))
@@
     (effects (font (size 1.27 1.27)) (justify left bottom))
   )
-  (label "GND10" (at 186.69 45.72 0) (fields_autoplaced)
+  (label "GND10" (at 186.69 50.8 0) (fields_autoplaced)
     (effects (font (size 1.27 1.27)) (justify left bottom))
   )
@@
     (effects (font (size 1.27 1.27)) (justify left bottom))
   )
-  (label "INP8" (at 166.37 22.86 0) (fields_autoplaced)
+  (label "INP8" (at 166.37 27.94 0) (fields_autoplaced)
     (effects (font (size 1.27 1.27)) (justify left bottom))
   )
-  (label "GND11" (at 186.69 50.8 0) (fields_autoplaced)
+  (label "GND11" (at 186.69 45.72 0) (fields_autoplaced)
     (effects (font (size 1.27 1.27)) (justify left bottom))
   )
@@
     (effects (font (size 1.27 1.27)) (justify left bottom))
   )
+  (label "VCC" (at 176.53 15.24 0) (fields_autoplaced)
+    (effects (font (size 1.27 1.27)) (justify left bottom))
+  )
   (label "GND3" (at 158.75 50.8 0) (fields_autoplaced)
     (effects (font (size 1.27 1.27)) (justify left bottom))
@@
     (effects (font (size 1.27 1.27)) (justify left bottom))
   )
-  (label "INP9" (at 166.37 27.94 0) (fields_autoplaced)
+  (label "INP9" (at 166.37 22.86 0) (fields_autoplaced)
     (effects (font (size 1.27 1.27)) (justify left bottom))
   )
@@
     (effects (font (size 1.27 1.27)) (justify left bottom))
   )
+  (label "VCC" (at 130.175 228.6 0) (fields_autoplaced)
+    (effects (font (size 1.27 1.27)) (justify left bottom))
+  )
   (label "GND6" (at 64.77 101.6 0) (fields_autoplaced)
     (effects (font (size 1.27 1.27)) (justify left bottom))
@@
     (effects (font (size 1.27 1.27)) (justify left bottom))
   )
+  (label "VCC" (at 148.59 83.82 0) (fields_autoplaced)
+    (effects (font (size 1.27 1.27)) (justify left bottom))
+  )
   (label "GND12" (at 110.49 168.91 0) (fields_autoplaced)
     (effects (font (size 1.27 1.27)) (justify left bottom))
@@
     (effects (font (size 1.27 1.27)) (justify left bottom))
   )
-  (label "INP14" (at 166.37 91.44 0) (fields_autoplaced)
+  (label "INP14" (at 166.37 96.52 0) (fields_autoplaced)
     (effects (font (size 1.27 1.27)) (justify left bottom))
   )
@@
     (effects (font (size 1.27 1.27)) (justify left bottom))
   )
-  (label "GND8" (at 186.69 22.86 0) (fields_autoplaced)
+  (label "GND8" (at 186.69 27.94 0) (fields_autoplaced)
     (effects (font (size 1.27 1.27)) (justify left bottom))
   )
@@
     (effects (font (size 1.27 1.27)) (justify left bottom))
   )
-  (label "INP12" (at 166.37 68.58 0) (fields_autoplaced)
+  (label "INP12" (at 166.37 73.66 0) (fields_autoplaced)
     (effects (font (size 1.27 1.27)) (justify left bottom))
   )
@@
     (effects (font (size 1.27 1.27)) (justify left bottom))
   )
-  (label "GND9" (at 186.69 27.94 0) (fields_autoplaced)
+  (label "GND9" (at 186.69 22.86 0) (fields_autoplaced)
     (effects (font (size 1.27 1.27)) (justify left bottom))
   )
@@
     (effects (font (size 1.27 1.27)) (justify left bottom))
   )
-  (label "INP11" (at 166.37 50.8 0) (fields_autoplaced)
+  (label "INP11" (at 166.37 45.72 0) (fields_autoplaced)
     (effects (font (size 1.27 1.27)) (justify left bottom))
   )
@@
     (effects (font (size 1.27 1.27)) (justify left bottom))
   )
+  (label "VCC" (at 176.53 38.1 0) (fields_autoplaced)
+    (effects (font (size 1.27 1.27)) (justify left bottom))
+  )
   (label "GND8" (at 80.01 120.65 0) (fields_autoplaced)
     (effects (font (size 1.27 1.27)) (justify left bottom))
@@
     (effects (font (size 1.27 1.27)) (justify left bottom))
   )
-  (label "INP13" (at 166.37 73.66 0) (fields_autoplaced)
+  (label "INP13" (at 166.37 68.58 0) (fields_autoplaced)
     (effects (font (size 1.27 1.27)) (justify left bottom))
   )
@@
     (effects (font (size 1.27 1.27)) (justify left bottom))
   )
+  (label "VCC" (at 176.53 83.82 0) (fields_autoplaced)
+    (effects (font (size 1.27 1.27)) (justify left bottom))
+  )
   (label "GND4" (at 64.77 74.93 0) (fields_autoplaced)
     (effects (font (size 1.27 1.27)) (justify left bottom))
@@
     (effects (font (size 1.27 1.27)) (justify left bottom))
   )
-  (label "INP10" (at 166.37 45.72 0) (fields_autoplaced)
+  (label "INP10" (at 166.37 50.8 0) (fields_autoplaced)
     (effects (font (size 1.27 1.27)) (justify left bottom))
   )
@@
     (effects (font (size 1.27 1.27)) (justify left bottom))
   )
+  (label "VCC" (at 148.59 38.1 0) (fields_autoplaced)
+    (effects (font (size 1.27 1.27)) (justify left bottom))
+  )
   (label "GND12" (at 64.77 168.91 0) (fields_autoplaced)
     (effects (font (size 1.27 1.27)) (justify left bottom))
   )
-  (label "GND12" (at 186.69 68.58 0) (fields_autoplaced)
+  (label "GND12" (at 186.69 73.66 0) (fields_autoplaced)
     (effects (font (size 1.27 1.27)) (justify left bottom))
   )
@@
     (effects (font (size 1.27 1.27)) (justify left bottom))
   )
+  (label "VCC" (at 148.59 60.96 0) (fields_autoplaced)
+    (effects (font (size 1.27 1.27)) (justify left bottom))
+  )
   (label "GND14" (at 95.25 193.04 0) (fields_autoplaced)
     (effects (font (size 1.27 1.27)) (justify left bottom))
@@
     (effects (font (size 1.27 1.27)) (justify left bottom))
   )
+  (label "VCC" (at 148.59 15.24 0) (fields_autoplaced)
+    (effects (font (size 1.27 1.27)) (justify left bottom))
+  )
   (label "GND" (at 148.59 58.42 0) (fields_autoplaced)
     (effects (font (size 1.27 1.27)) (justify left bottom))
@@
     (effects (font (size 1.27 1.27)) (justify left bottom))
   )
-  (label "INP15" (at 166.37 96.52 0) (fields_autoplaced)
+  (label "INP15" (at 166.37 91.44 0) (fields_autoplaced)
     (effects (font (size 1.27 1.27)) (justify left bottom))
   )
@@
     (effects (font (size 1.27 1.27)) (justify left bottom))
   )
-  (label "GND13" (at 186.69 73.66 0) (fields_autoplaced)
+  (label "GND13" (at 186.69 68.58 0) (fields_autoplaced)
     (effects (font (size 1.27 1.27)) (justify left bottom))
   )
@@
         )
       )
+    )
+  )
+  (symbol (lib_id "TacTile:Jumper_Connect") (at 130.175 228.6 0) (unit 1)
+    (in_bom yes) (on_board yes) (dnp no) (fields_autoplaced)
+    (property "Reference" "JMP17" (at 130.81 231.775 0)
+      (effects (font (size 1.27 1.27)) (justify left))
+    )
+    (property "Value" "~" (at 130.175 228.6 0)
+      (effects (font (size 1.27 1.27)))
+    )
+    (property "Footprint" "TacTile:Jumper_Connect" (at 130.175 228.6 0)
+      (effects (font (size 1.27 1.27)) hide)
+    )
+    (property "Datasheet" "" (at 130.175 228.6 0)
+      (effects (font (size 1.27 1.27)) hide)
+    )
+    (pin "1")
+    (instances
+      (project "TacTile-A"
+        (path "/6df59fdc-9f0d-414b-89c2-ac236518910e"
+          (reference "JMP17") (unit 1)
+        )
+      )
