File: TacTile-D/TacTile-D.kicad_sch (KiCad schematic)
At the start: 13 parts, among them J18 Conn_01x04, J18 Conn_01x06, J19 Conn_01x05, J19 Conn_01x06, J20 Conn_01x02, J20 Conn_01x06, J21 Conn_01x02, J21 Conn_01x06, U11 74LS04, U12 74HC595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

Commit message: Fixed counter clocking delay on D board
Parts:
- removed unit 2 of U11
Connections:
- net CLK: now also U13.13 (CPR); no longer U11.1
- net SEN: now also U11.1
- net at U12.13 (~{OE}), U13.14 (~{OE}): now also U11.2
- removed net ACLK: U11.2, U13.13 (CPR)
Other:
- moved on the sheet: U11A, U6A
